File: sim-hardware/flight-sim-radio/flight-sim-radio.kicad_sch (KiCad schematic)
At the start: 26 parts, among them J1 Conn_01x03, J2 Conn_01x09, J3 Conn_01x04, SW1 RS-08 300±150GF, SW2 RotaryEncoder_Switch, SW3 RotaryEncoder_Switch, U1 74LS148, U2 TM1637, U3 TM1637

Commit message: PCB checked
Parts:
- added R6, R7, R8, R9: 10k, Resistor_THT:R_Axial_DIN0207_L6.3mm_D2.5mm_P10.16mm_Horizontal, symbol Device:R
Connections:
- net D1_CLK: now also R6.1
- net D1_DIO: now also R7.1
- net D2_CLK: now also R8.1
- net D2_DIO: now also R9.1
- net VDD: now also R6.2, R7.2, R8.2, R9.2
